Commit message: initial commit

File: living_lab_robot_description/urdf/mobile_assy.urdf.xacro (robot description, xacro)
@@ -16,7 +16,7 @@
         </collision>
         <inertial>
-            <origin xyz="0 0 0" rpy="0 0 0"/>
-            <mass value="30.0"/>
-            <inertia ixx="10.0" ixy="0.0" ixz="0.0" iyy="10.0" iyz="0.0" izz="10.0"/>
+            <origin xyz="0 0 0.1111" rpy="0 0 0"/>
+            <mass value="55.0"/>
+            <inertia ixx="1.700489" ixy="0.0" ixz="0.0" iyy="1.700489" iyz="0.0" izz="2.604803"/>
         </inertial>
     </link>
@@ -27,9 +27,9 @@
     </joint>
     <link name="front_hokuyo_link">
-        <inertial>
+        <!-- <inertial>
             <origin xyz="0 0 0" rpy="0 0 0"/>
             <mass value="1.0"/>
             <inertia ixx="1.0" ixy="0.0" ixz="0.0" iyy="1.0" iyz="0.0" izz="1.0"/>
-        </inertial>
+        </inertial> -->
     </link>
     <xacro:insert_hokuyo_sensor name="front" />
@@ -40,9 +40,9 @@
     </joint>
     <link name="rear_hokuyo_link">
-        <inertial>
+        <!-- <inertial>
             <origin xyz="0 0 0" rpy="0 0 0"/>
             <mass value="1.0"/>
             <inertia ixx="1.0" ixy="0.0" ixz="0.0" iyy="1.0" iyz="0.0" izz="1.0"/>
-        </inertial>
+        </inertial> -->
     </link>
     <xacro:insert_hokuyo_sensor name="rear" />
@@ -62,11 +62,11 @@
             <origin xyz="0 0 0" rpy="0 0 0"/>
             <geometry>
-                <mesh filename="package://living_lab_robot_description/meshes/omni_wheel.dae" scale="1 1 1"/>
+                <sphere radius="0.065"/>
             </geometry>
         </collision>
         <inertial>
-            <origin xyz="0 0 0" rpy="0 0 0"/>
-            <mass value="1.0"/>
-            <inertia ixx="1.0" ixy="0.0" ixz="0.0" iyy="1.0" iyz="0.0" izz="1.0"/>
+            <origin xyz="0 -0.0015 0" rpy="0 0 0"/>
+            <mass value="0.42"/>
+            <inertia ixx="0.000562" ixy="0.0" ixz="0.0" iyy="0.000884" iyz="0.0" izz="0.000562"/>
         </inertial>
     </link>
@@ -88,11 +88,11 @@
             <origin xyz="0 0 0" rpy="0 0 0"/>
             <geometry>
-                <mesh filename="package://living_lab_robot_description/meshes/omni_wheel.dae" scale="1 1 1"/>
+                <sphere radius="0.065"/>
             </geometry>
         </collision>
         <inertial>
-            <origin xyz="0 0 0" rpy="0 0 0"/>
-            <mass value="1.0"/>
-            <inertia ixx="1.0" ixy="0.0" ixz="0.0" iyy="1.0" iyz="0.0" izz="1.0"/>
+            <origin xyz="0 -0.0015 0" rpy="0 0 0"/>
+            <mass value="0.42"/>
+            <inertia ixx="0.000562" ixy="0.0" ixz="0.0" iyy="0.000884" iyz="0.0" izz="0.000562"/>
         </inertial>
     </link>
@@ -114,11 +114,11 @@
             <origin xyz="0 0 0" rpy="0 0 0"/>
             <geometry>
-                <mesh filename="package://living_lab_robot_description/meshes/omni_wheel.dae" scale="1 1 1"/>
+                <sphere radius="0.065"/>
             </geometry>
         </collision>
         <inertial>
-            <origin xyz="0 0 0" rpy="0 0 0"/>
-            <mass value="1.0"/>
-            <inertia ixx="1.0" ixy="0.0" ixz="0.0" iyy="1.0" iyz="0.0" izz="1.0"/>
+            <origin xyz="0 -0.0015 0" rpy="0 0 0"/>
+            <mass value="0.42"/>
+            <inertia ixx="0.000562" ixy="0.0" ixz="0.0" iyy="0.000884" iyz="0.0" izz="0.000562"/>
         </inertial>
     </link>

File: living_lab_robot_description/urdf/robot.urdf.xacro (robot description, xacro)
@@ -7,4 +7,7 @@
     <xacro:include filename="$(find living_lab_robot_description)/urdf/arm.urdf.xacro"/>
     <xacro:include filename="$(find living_lab_robot_description)/urdf/gripper.urdf.xacro"/>
+    <robotis_gripper parent="arm_link6">
+        <origin xyz="0 0 0" rpy="0 0 0"/>
+    </robotis_gripper>
     <xacro:include filename="$(find living_lab_robot_description)/urdf/head_assy.urdf.xacro"/>
 </robot>
